Commit message: Run the rover in Gazebo Harmonic alongside Classic.
Adds a Jazzy/Harmonic Docker image, a sim:=harmonic option in the rover xacro (default output unchanged), gz_harmonic.launch.py, a ros_gz bridge keeping the Classic topic names, Jazzy controller settings, and a Twist to TwistStamped converter.

Co-authored-by: Cursor <cursoragent@cursor.com>

File: src/four_wheel_sim/urdf/robot.urdf.xacro (robot description, xacro)
@@ -1,4 +1,7 @@
 <?xml version="1.0"?>
 <robot name="four_wheel_bot" xmlns:xacro="http://www.ros.org/wiki/xacro">
+  <!-- classic: Gazebo Classic 11 on Humble. harmonic: Gazebo Harmonic on Jazzy. -->
+  <xacro:arg name="sim" default="classic"/>
+  <xacro:property name="classic" value="${'$(arg sim)' == 'classic'}"/>
   <material name="blue"><color rgba="0.2 0.4 0.8 1"/></material>
   <material name="black"><color rgba="0.1 0.1 0.1 1"/></material>
@@ -14,5 +17,7 @@
     </inertial>
   </link>
-  <gazebo reference="base_link"><material>Gazebo/Blue</material></gazebo>
+  <xacro:if value="${classic}">
+    <gazebo reference="base_link"><material>Gazebo/Blue</material></gazebo>
+  </xacro:if>
   <xacro:macro name="wheel" params="name x y">
     <link name="${name}_wheel">
@@ -39,5 +44,5 @@
       <mu1>0.9</mu1><mu2>0.8</mu2>
       <fdir1>1 0 0</fdir1>
-      <material>Gazebo/Black</material>
+      <xacro:if value="${classic}"><material>Gazebo/Black</material></xacro:if>
       <minDepth>0.001</minDepth>
       <kp>1e6</kp><kd>100</kd>
@@ -49,5 +54,8 @@
   <xacro:wheel name="rear_right"  x="-0.13" y="-0.12"/>
   <ros2_control name="GazeboSystem" type="system">
-    <hardware><plugin>gazebo_ros2_control/GazeboSystem</plugin></hardware>
+    <hardware>
+      <xacro:if value="${classic}"><plugin>gazebo_ros2_control/GazeboSystem</plugin></xacro:if>
+      <xacro:unless value="${classic}"><plugin>gz_ros2_control/GazeboSimSystem</plugin></xacro:unless>
+    </hardware>
     <joint name="front_left_wheel_joint">
       <command_interface name="velocity"><param name="min">-20</param><param name="max">20</param></command_interface>
@@ -67,18 +75,35 @@
     </joint>
   </ros2_control>
-  <gazebo>
-    <plugin name="gazebo_ros2_control" filename="libgazebo_ros2_control.so">
-      <parameters>$(find four_wheel_sim)/config/controllers.yaml</parameters>
-    </plugin>
-    <plugin name="ground_truth" filename="libgazebo_ros_p3d.so">
-      <ros><remapping>odom:=odom_gt</remapping></ros>
-      <body_name>base_link</body_name>
-      <frame_name>world</frame_name>
-      <update_rate>50.0</update_rate>
-      <xyz_offset>0 0 0</xyz_offset>
-      <rpy_offset>0 0 0</rpy_offset>
-      <gaussian_noise>0.0</gaussian_noise>
-    </plugin>
-  </gazebo>
+  <xacro:if value="${classic}">
+    <gazebo>
+      <plugin name="gazebo_ros2_control" filename="libgazebo_ros2_control.so">
+        <parameters>$(find four_wheel_sim)/config/controllers.yaml</parameters>
+      </plugin>
+      <plugin name="ground_truth" filename="libgazebo_ros_p3d.so">
+        <ros><remapping>odom:=odom_gt</remapping></ros>
+        <body_name>base_link</body_name>
+        <frame_name>world</frame_name>
+        <update_rate>50.0</update_rate>
+        <xyz_offset>0 0 0</xyz_offset>
+        <rpy_offset>0 0 0</rpy_offset>
+        <gaussian_noise>0.0</gaussian_noise>
+      </plugin>
+    </gazebo>
+  </xacro:if>
+  <xacro:unless value="${classic}">
+    <gazebo>
+      <plugin name="gz_ros2_control::GazeboSimROS2ControlPlugin" filename="gz_ros2_control-system">
+        <parameters>$(find four_wheel_sim)/config/controllers_jazzy.yaml</parameters>
+      </plugin>
+      <!-- World-frame pose of base_link, bridged to ROS as /odom_gt. -->
+      <plugin name="gz::sim::systems::OdometryPublisher" filename="gz-sim-odometry-publisher-system">
+        <odom_frame>world</odom_frame>
+        <robot_base_frame>base_link</robot_base_frame>
+        <odom_topic>/odom_gt</odom_topic>
+        <odom_publish_frequency>50</odom_publish_frequency>
+        <dimensions>3</dimensions>
+      </plugin>
+    </gazebo>
+  </xacro:unless>
   <link name="camera_link">
     <visual>
@@ -100,20 +125,40 @@
     <origin rpy="-1.5708 0 -1.5708"/>
   </joint>
-  <gazebo reference="camera_link">
-    <sensor name="oak_d" type="depth">
-      <always_on>true</always_on>
-      <update_rate>15</update_rate>
-      <camera>
-        <horizontal_fov>1.22</horizontal_fov>
-        <image><width>640</width><height>400</height><format>R8G8B8</format></image>
-        <clip><near>0.3</near><far>8.0</far></clip>
-      </camera>
-      <plugin name="oak_d_plugin" filename="libgazebo_ros_camera.so">
-        <camera_name>oak</camera_name>
-        <frame_name>camera_optical_frame</frame_name>
-        <min_depth>0.3</min_depth>
-        <max_depth>8.0</max_depth>
-      </plugin>
-    </sensor>
-  </gazebo>
+  <xacro:if value="${classic}">
+    <gazebo reference="camera_link">
+      <sensor name="oak_d" type="depth">
+        <always_on>true</always_on>
+        <update_rate>15</update_rate>
+        <camera>
+          <horizontal_fov>1.22</horizontal_fov>
+          <image><width>640</width><height>400</height><format>R8G8B8</format></image>
+          <clip><near>0.3</near><far>8.0</far></clip>
+        </camera>
+        <plugin name="oak_d_plugin" filename="libgazebo_ros_camera.so">
+          <camera_name>oak</camera_name>
+          <frame_name>camera_optical_frame</frame_name>
+          <min_depth>0.3</min_depth>
+          <max_depth>8.0</max_depth>
+        </plugin>
+      </sensor>
+    </gazebo>
+  </xacro:if>
+  <xacro:unless value="${classic}">
+    <!-- Publishes oak/image, oak/depth_image, oak/camera_info, and oak/points in
+         Gazebo. config/gz_bridge.yaml maps them to the Classic ROS topic names. -->
+    <gazebo reference="camera_link">
+      <sensor name="oak_d" type="rgbd_camera">
+        <always_on>true</always_on>
+        <update_rate>15</update_rate>
+        <topic>oak</topic>
+        <gz_frame_id>camera_optical_frame</gz_frame_id>
+        <camera>
+          <horizontal_fov>1.22</horizontal_fov>
+          <image><width>640</width><height>400</height><format>R8G8B8</format></image>
+          <clip><near>0.3</near><far>8.0</far></clip>
+          <depth_camera><clip><near>0.3</near><far>8.0</far></clip></depth_camera>
+        </camera>
+      </sensor>
+    </gazebo>
+  </xacro:unless>
 </robot>

Commit message: Raise the camera to 1080p at 30 in and add Mars sampling-site analogues.
The camera now captures 1920x1080 RGB at 30 Hz with its optical center 0.762 m
above level ground. The mount is 0.682 m above base_link because base_link rests
0.08 m off the ground. A visual mast fills the gap. The FOV stays 1.22 rad and is
marked provisional. The runtime check verifies size, rate, intrinsics, and height.

Scenes can now include silica-like soil patches, fractured sulfur-bearing stones,
and Cheyava-like veined, spotted mudstone slabs, each with a lookalike control.
They are visual analogues built from NASA reference photos, not copies of them.
Labels carry seven classes. Ground patches also get a mask.

Co-authored-by: Cursor <cursoragent@cursor.com>

File: src/four_wheel_sim/urdf/robot.urdf.xacro (robot description, xacro)
@@ -7,7 +7,15 @@
   <material name="black"><color rgba="0.1 0.1 0.1 1"/></material>
   <link name="base_link">
-    <visual>
+    <visual name="chassis">
       <geometry><box size="0.4 0.2 0.1"/></geometry>
       <material name="blue"/>
+    </visual>
+    <!-- Visual only. No collision, so the mast does not change driving.
+         The post runs from the chassis top (z = 0.05) to the camera origin
+         (z = 0.682). See the camera_joint comment for that height. -->
+    <visual name="camera_mast">
+      <origin xyz="0.2 0 0.366" rpy="0 0 0"/>
+      <geometry><box size="0.02 0.02 0.632"/></geometry>
+      <material name="black"/>
     </visual>
     <collision><geometry><box size="0.4 0.2 0.1"/></geometry></collision>
@@ -116,7 +124,15 @@
     </inertial>
   </link>
+  <!-- Wheel spheres of radius 0.05 m are centered 0.03 m below base_link, so
+       the origin rests 0.08 m above level ground. The optical frame has no
+       translation from camera_link, so this joint Z is the optical center in
+       base_link, not the height above the ground.
+       30 in = 0.762 m above the contact plane => z = 0.762 - 0.08 = 0.682.
+       Pitch 0.1 rad noses the body, sensor, and optical frame down together.
+       horizontal_fov 1.22 rad below is provisional, not a measured OAK-D
+       calibration. The RGB-D sensor has one image size, so depth follows RGB. -->
   <joint name="camera_joint" type="fixed">
     <parent link="base_link"/><child link="camera_link"/>
-    <origin xyz="0.2 0 0.12" rpy="0 0.1 0"/>
+    <origin xyz="0.2 0 0.682" rpy="0 0.1 0"/>
   </joint>
   <link name="camera_optical_frame"/>
@@ -129,8 +145,8 @@
       <sensor name="oak_d" type="depth">
         <always_on>true</always_on>
-        <update_rate>15</update_rate>
+        <update_rate>30</update_rate>
         <camera>
           <horizontal_fov>1.22</horizontal_fov>
-          <image><width>640</width><height>400</height><format>R8G8B8</format></image>
+          <image><width>1920</width><height>1080</height><format>R8G8B8</format></image>
           <clip><near>0.3</near><far>8.0</far></clip>
         </camera>
@@ -150,10 +166,10 @@
       <sensor name="oak_d" type="rgbd_camera">
         <always_on>true</always_on>
-        <update_rate>15</update_rate>
+        <update_rate>30</update_rate>
         <topic>oak</topic>
         <gz_frame_id>camera_optical_frame</gz_frame_id>
         <camera>
           <horizontal_fov>1.22</horizontal_fov>
-          <image><width>640</width><height>400</height><format>R8G8B8</format></image>
+          <image><width>1920</width><height>1080</height><format>R8G8B8</format></image>
           <clip><near>0.3</near><far>8.0</far></clip>
           <depth_camera><clip><near>0.3</near><far>8.0</far></clip></depth_camera>
