Commit message: Switched control scheme over to Nav2 ros package

File: src/four_wheel_sim/urdf/robot.urdf.xacro (robot description, xacro)
@@ -36,6 +36,8 @@
     </joint>
     <gazebo reference="${name}_wheel">
-      <mu1>1.0</mu1><mu2>0.1</mu2>
+      <mu1>0.6</mu1><mu2>0.6</mu2>
       <material>Gazebo/Black</material>
+      <minDepth>0.001</minDepth>
+      <kp>1e6</kp><kd>100</kd>
     </gazebo>
   </xacro:macro>
@@ -44,29 +46,26 @@
   <xacro:wheel name="front_right" x="0.13"  y="-0.12"/>
   <xacro:wheel name="rear_right"  x="-0.13" y="-0.12"/>
+  <ros2_control name="GazeboSystem" type="system">
+    <hardware><plugin>gazebo_ros2_control/GazeboSystem</plugin></hardware>
+    <joint name="front_left_wheel_joint">
+      <command_interface name="velocity"><param name="min">-20</param><param name="max">20</param></command_interface>
+      <state_interface name="position"/><state_interface name="velocity"/>
+    </joint>
+    <joint name="rear_left_wheel_joint">
+      <command_interface name="velocity"><param name="min">-20</param><param name="max">20</param></command_interface>
+      <state_interface name="position"/><state_interface name="velocity"/>
+    </joint>
+    <joint name="front_right_wheel_joint">
+      <command_interface name="velocity"><param name="min">-20</param><param name="max">20</param></command_interface>
+      <state_interface name="position"/><state_interface name="velocity"/>
+    </joint>
+    <joint name="rear_right_wheel_joint">
+      <command_interface name="velocity"><param name="min">-20</param><param name="max">20</param></command_interface>
+      <state_interface name="position"/><state_interface name="velocity"/>
+    </joint>
+  </ros2_control>
   <gazebo>
-    <plugin name="diff_drive" filename="libgazebo_ros_diff_drive.so">
-      <update_rate>50</update_rate>
-      <num_wheel_pairs>2</num_wheel_pairs>
-      <left_joint>front_left_wheel_joint</left_joint>
-      <right_joint>front_right_wheel_joint</right_joint>
-      <left_joint>rear_left_wheel_joint</left_joint>
-      <right_joint>rear_right_wheel_joint</right_joint>
-      <wheel_separation>0.24</wheel_separation>
-      <wheel_separation>0.24</wheel_separation>
-      <wheel_diameter>0.1</wheel_diameter>
-      <wheel_diameter>0.1</wheel_diameter>
-      <max_wheel_torque>20</max_wheel_torque>
-      <max_wheel_acceleration>3.0</max_wheel_acceleration>
-      <odometry_frame>odom</odometry_frame>
-      <robot_base_frame>base_link</robot_base_frame>
-      <publish_odom>true</publish_odom>
-      <publish_odom_tf>true</publish_odom_tf>
-    </plugin>
-    <plugin name="joint_states" filename="libgazebo_ros_joint_state_publisher.so">
-      <update_rate>30</update_rate>
-      <joint_name>front_left_wheel_joint</joint_name>
-      <joint_name>rear_left_wheel_joint</joint_name>
-      <joint_name>front_right_wheel_joint</joint_name>
-      <joint_name>rear_right_wheel_joint</joint_name>
+    <plugin name="gazebo_ros2_control" filename="libgazebo_ros2_control.so">
+      <parameters>$(find four_wheel_sim)/config/controllers.yaml</parameters>
     </plugin>
   </gazebo>

Commit message: Had to change the odomtry topic due to conflicts. Changed wheels in sim to be spheres instead of cylinders for future testing.

File: src/four_wheel_sim/urdf/robot.urdf.xacro (robot description, xacro)
@@ -23,6 +23,5 @@
       </visual>
       <collision>
-        <origin rpy="1.5708 0 0"/>
-        <geometry><cylinder radius="0.05" length="0.04"/></geometry>
+        <geometry><sphere radius="0.05"/></geometry>
       </collision>
       <inertial>
@@ -34,7 +33,10 @@
       <parent link="base_link"/><child link="${name}_wheel"/>
       <origin xyz="${x} ${y} -0.03"/><axis xyz="0 1 0"/>
+      <limit effort="10" velocity="20"/>
+      <dynamics damping="0.0" friction="0.0"/>
     </joint>
     <gazebo reference="${name}_wheel">
-      <mu1>0.6</mu1><mu2>0.6</mu2>
+      <mu1>1.0</mu1><mu2>0.30</mu2>
+      <fdir1>1 0 0</fdir1>
       <material>Gazebo/Black</material>
       <minDepth>0.001</minDepth>
@@ -69,4 +71,13 @@
       <parameters>$(find four_wheel_sim)/config/controllers.yaml</parameters>
     </plugin>
+    <plugin name="ground_truth" filename="libgazebo_ros_p3d.so">
+      <ros><remapping>odom:=odom_gt</remapping></ros>
+      <body_name>base_link</body_name>
+      <frame_name>world</frame_name>
+      <update_rate>50.0</update_rate>
+      <xyz_offset>0 0 0</xyz_offset>
+      <rpy_offset>0 0 0</rpy_offset>
+      <gaussian_noise>0.0</gaussian_noise>
+    </plugin>
   </gazebo>
 </robot>

Commit message: Added basic RGB and Depth camera into Gazebo simulation for testing.

File: src/four_wheel_sim/urdf/robot.urdf.xacro (robot description, xacro)
@@ -37,5 +37,5 @@
     </joint>
     <gazebo reference="${name}_wheel">
-      <mu1>1.0</mu1><mu2>0.30</mu2>
+      <mu1>0.9</mu1><mu2>0.9</mu2>
       <fdir1>1 0 0</fdir1>
       <material>Gazebo/Black</material>
@@ -81,3 +81,39 @@
     </plugin>
   </gazebo>
+  <link name="camera_link">
+    <visual>
+      <geometry><box size="0.03 0.09 0.03"/></geometry>
+      <material name="black"/>
+    </visual>
+    <inertial>
+      <mass value="0.1"/>
+      <inertia ixx="0.0001" iyy="0.0001" izz="0.0001" ixy="0" ixz="0" iyz="0"/>
+    </inertial>
+  </link>
+  <joint name="camera_joint" type="fixed">
+    <parent link="base_link"/><child link="camera_link"/>
+    <origin xyz="0.2 0 0.08"/>
+  </joint>
+  <link name="camera_optical_frame"/>
+  <joint name="camera_optical_joint" type="fixed">
+    <parent link="camera_link"/><child link="camera_optical_frame"/>
+    <origin rpy="-1.5708 0 -1.5708"/>
+  </joint>
+  <gazebo reference="camera_link">
+    <sensor name="oak_d" type="depth">
+      <always_on>true</always_on>
+      <update_rate>15</update_rate>
+      <camera>
+        <horizontal_fov>1.22</horizontal_fov>
+        <image><width>640</width><height>400</height><format>R8G8B8</format></image>
+        <clip><near>0.3</near><far>8.0</far></clip>
+      </camera>
+      <plugin name="oak_d_plugin" filename="libgazebo_ros_camera.so">
+        <camera_name>oak</camera_name>
+        <frame_name>camera_optical_frame</frame_name>
+        <min_depth>0.3</min_depth>
+        <max_depth>8.0</max_depth>
+      </plugin>
+    </sensor>
+  </gazebo>
 </robot>

Commit message: Changed urdf file so that path planning runs on AStar path planning algo. Will test on a determined maze

File: src/four_wheel_sim/urdf/robot.urdf.xacro (robot description, xacro)
@@ -37,5 +37,5 @@
     </joint>
     <gazebo reference="${name}_wheel">
-      <mu1>0.9</mu1><mu2>0.9</mu2>
+      <mu1>0.9</mu1><mu2>0.8</mu2>
       <fdir1>1 0 0</fdir1>
       <material>Gazebo/Black</material>
@@ -93,5 +93,5 @@
   <joint name="camera_joint" type="fixed">
     <parent link="base_link"/><child link="camera_link"/>
-    <origin xyz="0.2 0 0.08"/>
+    <origin xyz="0.2 0 0.12" rpy="0 0.1 0"/>
   </joint>
   <link name="camera_optical_frame"/>

Commit message: Attempting to switch map over to a more flat terrain like it will actually be used.

File: src/four_wheel_sim/urdf/robot.urdf.xacro (robot description, xacro)
@@ -66,4 +66,8 @@
       <state_interface name="position"/><state_interface name="velocity"/>
     </joint>
+    <joint name="head_pan_joint">
+      <command_interface name="position"/>
+      <state_interface name="position"/><state_interface name="velocity"/>
+    </joint>
   </ros2_control>
   <gazebo>
@@ -91,7 +95,23 @@
     </inertial>
   </link>
+  <link name="head_link">
+    <visual>
+      <geometry><cylinder radius="0.04" length="0.04"/></geometry>
+      <material name="black"/>
+    </visual>
+    <inertial>
+      <mass value="0.2"/>
+      <inertia ixx="0.0002" iyy="0.0002" izz="0.0002" ixy="0" ixz="0" iyz="0"/>
+    </inertial>
+  </link>
+  <joint name="head_pan_joint" type="continuous">
+    <parent link="base_link"/><child link="head_link"/>
+    <origin xyz="0 0 0.1"/><axis xyz="0 0 1"/>
+    <limit effort="5" velocity="2.0"/>
+    <dynamics damping="0.1"/>
+  </joint>
   <joint name="camera_joint" type="fixed">
-    <parent link="base_link"/><child link="camera_link"/>
-    <origin xyz="0.2 0 0.12" rpy="0 0.1 0"/>
+    <parent link="head_link"/><child link="camera_link"/>
+    <origin xyz="0.05 0 0.03" rpy="0 0.2 0"/>
   </joint>
   <link name="camera_optical_frame"/>
