Commit message: Added mesh for better visuals

File: arm_description/urdf/arm.urdf.xacro (robot description, xacro)
@@ -1,115 +1,487 @@
-<?xml version="1.0"?>
-<robot name="six_servo_arm" xmlns:xacro="http://www.ros.org/wiki/xacro">
-  <!-- Placeholder dimensions, in meters -->
-  <xacro:property name="base_h" value="0.06"/>
-  <xacro:property name="upper_arm" value="0.12"/>
-  <xacro:property name="forearm" value="0.12"/>
-  <xacro:property name="wrist_len" value="0.06"/>
-  <!-- Reusable visual link -->
-  <xacro:macro name="arm_link" params="name length radius">
-    <link name="${name}">
-      <visual>
-        <origin xyz="0 0 ${length/2}" rpy="0 0 0"/>
-        <geometry>
-          <cylinder radius="${radius}" length="${length}"/>
-        </geometry>
-        <material name="arm_blue">
-          <color rgba="0.2 0.4 0.8 1"/>
-        </material>
-      </visual>
-      <collision>
-        <origin xyz="0 0 ${length/2}"/>
-        <geometry>
-          <cylinder radius="${radius}" length="${length}"/>
-        </geometry>
-      </collision>
-      <inertial>
-        <origin xyz="0 0 ${length/2}"/>
-        <mass value="0.2"/>
-        <inertia ixx="0.001" ixy="0" ixz="0"
-                 iyy="0.001" iyz="0" izz="0.001"/>
-      </inertial>
-    </link>
-  </xacro:macro>
-  <!-- Base -->
+<?xml version="1.0" encoding="utf-8"?>
+<!-- This URDF was automatically created by SolidWorks to URDF Exporter! Originally created by Stephen Brawner (brawner@gmail.com)
+     Commit Version: 1.6.0-4-g7f85cfe  Build Version: 1.6.7995.38578
+     For more information, please see http://wiki.ros.org/sw_urdf_exporter -->
+<robot
+  name="arm_description">
   <link name="base_link">
-    <visual>
-      <geometry>
-        <cylinder radius="0.055" length="${base_h}"/>
-      </geometry>
-      <material name="base_gray">
-        <color rgba="0.35 0.35 0.35 1"/>
-      </material>
-    </visual>
-    <collision>
-      <geometry>
-        <cylinder radius="0.055" length="${base_h}"/>
-      </geometry>
-    </collision>
-    <inertial>
-      <mass value="1.0"/>
-      <inertia ixx="0.002" ixy="0" ixz="0"
-               iyy="0.002" iyz="0" izz="0.002"/>
-    </inertial>
-  </link>
-  <!-- Servo 1: base rotation -->
-  <link name="shoulder_mount">
-    <visual>
-      <geometry><cylinder radius="0.035" length="0.04"/></geometry>
-      <material name="joint_gray">
-        <color rgba="0.5 0.5 0.5 1"/></material>
-    </visual>
-  </link>
-  <joint name="base_yaw" type="revolute">
-    <parent link="base_link"/>
-    <child link="shoulder_mount"/>
-    <origin xyz="0 0 ${base_h/2}" rpy="0 0 0"/>
-    <axis xyz="0 0 1"/>
-    <limit lower="-2.35" upper="2.35" effort="5" velocity="1.0"/>
-  </joint>
-  <!-- Servo 2: shoulder pitch -->
-  <xacro:arm_link name="upper_arm_link" length="${upper_arm}" radius="0.018"/>
-  <joint name="shoulder_pitch" type="revolute">
-    <parent link="shoulder_mount"/>
-    <child link="upper_arm_link"/>
-    <origin xyz="0 0 0.02" rpy="0 0 0"/>
-    <axis xyz="0 1 0"/>
-    <limit lower="-1.57" upper="1.57" effort="5" velocity="1.0"/>
-  </joint>
-  <!-- Servo 3: elbow pitch -->
-  <xacro:arm_link name="forearm_link" length="${forearm}" radius="0.015"/>
-  <joint name="elbow_pitch" type="revolute">
-    <parent link="upper_arm_link"/>
-    <child link="forearm_link"/>
-    <origin xyz="0 0 ${upper_arm}" rpy="0 0 0"/>
-    <axis xyz="0 1 0"/>
-    <limit lower="-2.0" upper="2.0" effort="5" velocity="1.0"/>
-  </joint>
-  <!-- Servo 4: wrist pitch -->
-  <xacro:arm_link name="wrist_pitch_link" length="${wrist_len}" radius="0.012"/>
-  <joint name="wrist_pitch" type="revolute">
-    <parent link="forearm_link"/>
-    <child link="wrist_pitch_link"/>
-    <origin xyz="0 0 ${forearm}" rpy="0 0 0"/>
-    <axis xyz="0 1 0"/>
-    <limit lower="-1.57" upper="1.57" effort="3" velocity="1.0"/>
-  </joint>
-  <!-- Servo 5: wrist rotation -->
-  <link name="gripper_mount"/>
-  <joint name="wrist_roll" type="revolute">
-    <parent link="wrist_pitch_link"/>
-    <child link="gripper_mount"/>
-    <origin xyz="0 0 ${wrist_len}" rpy="0 0 0"/>
-    <axis xyz="0 0 1"/>
-    <limit lower="-2.35" upper="2.35" effort="3" velocity="1.0"/>
-  </joint>
-  <!-- Servo 6: gripper opening -->
-  <xacro:arm_link name="gripper_finger" length="0.05" radius="0.005"/>
-  <joint name="gripper" type="revolute">
-    <parent link="gripper_mount"/>
-    <child link="gripper_finger"/>
-    <origin xyz="0 0 0.025" rpy="0 0 0"/>
-    <axis xyz="1 0 0"/>
-    <limit lower="0" upper="0.7" effort="2" velocity="1.0"/>
+   </link>
+  <joint name="Base_joint" type="fixed">
+     <parent link="base_link"/>
+     <child link="Link_0"/>
+   </joint>
+  <link
+    name="Link_0">
+    <inertial>
+      <origin
+        xyz="-0.00186841174166371 2.50538852245872E-08 0.0215517174968573"
+        rpy="0 0 0" />
+      <mass
+        value="0.120274881687953" />
+      <inertia
+        ixx="7.85095489782459E-05"
+        ixy="-2.5923964914073E-10"
+        ixz="7.52479004938925E-07"
+        iyy="5.40736714848378E-05"
+        iyz="-1.15213465229022E-10"
+        izz="0.000105809384793902" />
+    </inertial>
+    <visual>
+      <origin
+        xyz="0 0 0"
+        rpy="0 0 0" />
+      <geometry>
+        <mesh
+          filename="package://arm_description/meshes/Link_0.STL" />
+      </geometry>
+      <material
+        name="">
+        <color
+          rgba="0.752941176470588 0.752941176470588 0.752941176470588 1" />
+      </material>
+    </visual>
+    <collision>
+      <origin
+        xyz="0 0 0"
+        rpy="0 0 0" />
+      <geometry>
+        <mesh
+          filename="package://arm_description/meshes/Link_0.STL" />
+      </geometry>
+    </collision>
+  </link>
+  <link
+    name="Link_1">
+    <inertial>
+      <origin
+        xyz="1.6372825671052E-08 -0.00192246981351583 0.0249618879819944"
+        rpy="0 0 0" />
+      <mass
+        value="0.0601843511838218" />
+      <inertia
+        ixx="2.40354508371122E-05"
+        ixy="7.39479891402167E-12"
+        ixz="2.05889155998936E-11"
+        iyy="2.50929356191337E-05"
+        iyz="-2.8998043123432E-07"
+        izz="1.79760286790951E-05" />
+    </inertial>
+    <visual>
+      <origin
+        xyz="0 0 0"
+        rpy="0 0 0" />
+      <geometry>
+        <mesh
+          filename="package://arm_description/meshes/Link_1.STL" />
+      </geometry>
+      <material
+        name="">
+        <color
+          rgba="0.752941176470588 0.752941176470588 0.752941176470588 1" />
+      </material>
+    </visual>
+    <collision>
+      <origin
+        xyz="0 0 0"
+        rpy="0 0 0" />
+      <geometry>
+        <mesh
+          filename="package://arm_description/meshes/Link_1.STL" />
+      </geometry>
+    </collision>
+  </link>
+  <joint
+    name="Joint_1"
+    type="revolute">
+    <origin
+      xyz="0 0 0.0520999749999999"
+      rpy="0 0 0" />
+    <parent
+      link="Link_0" />
+    <child
+      link="Link_1" />
+    <axis
+      xyz="0 0 1" />
+    <limit
+      lower="-3.14"
+      upper="3.14"
+      effort="2.92"
+      velocity="4.5" />
+  </joint>
+  <link
+    name="Link_2">
+    <inertial>
+      <origin
+        xyz="0.00639934747655226 -0.000788371670941635 0.0673431569215511"
+        rpy="0 0 0" />
+      <mass
+        value="0.0879365609479581" />
+      <inertia
+        ixx="5.58125584142004E-05"
+        ixy="3.05873895421976E-07"
+        ixz="-6.11348651523486E-07"
+        iyy="5.08744603129432E-05"
+        iyz="2.78428454591459E-07"
+        izz="2.91228934054131E-05" />
+    </inertial>
+    <visual>
+      <origin
+        xyz="0 0 0"
+        rpy="0 0 0" />
+      <geometry>
+        <mesh
+          filename="package://arm_description/meshes/Link_2.STL" />
+      </geometry>
+      <material
+        name="">
+        <color
+          rgba="0.752941176470588 0.752941176470588 0.752941176470588 1" />
+      </material>
+    </visual>
+    <collision>
+      <origin
+        xyz="0 0 0"
+        rpy="0 0 0" />
+      <geometry>
+        <mesh
+          filename="package://arm_description/meshes/Link_2.STL" />
+      </geometry>
+    </collision>
+  </link>
+  <joint
+    name="Joint_2"
+    type="revolute">
+    <origin
+      xyz="0 0 0.0541000250000002"
+      rpy="0 0 0" />
+    <parent
+      link="Link_1" />
+    <child
+      link="Link_2" />
+    <axis
+      xyz="0 1 0" />
+    <limit
+      lower="-1.57"
+      upper="1.57"
+      effort="2.94"
+      velocity="4.5" />
+  </joint>
+  <link
+    name="Link_3">
+    <inertial>
+      <origin
+        xyz="0.0717174331065269 -0.000795514048423572 0.000196159539195329"
+        rpy="0 0 0" />
+      <mass
+        value="0.0879996844183864" />
+      <inertia
+        ixx="2.19988198885556E-05"
+        ixy="5.11334783735054E-07"
+        ixz="-2.57342143473836E-08"
+        iyy="5.13996982896891E-05"
+        iyz="5.45466342941832E-11"
+        izz="6.34682921546949E-05" />
+    </inertial>
+    <visual>
+      <origin
+        xyz="0 0 0"
+        rpy="0 0 0" />
+      <geometry>
+        <mesh
+          filename="package://arm_description/meshes/Link_3.STL" />
+      </geometry>
+      <material
+        name="">
+        <color
+          rgba="0.752941176470588 0.752941176470588 0.752941176470588 1" />
+      </material>
+    </visual>
+    <collision>
+      <origin
+        xyz="0 0 0"
+        rpy="0 0 0" />
+      <geometry>
+        <mesh
+          filename="package://arm_description/meshes/Link_3.STL" />
+      </geometry>
+    </collision>
+  </link>
+  <joint
+    name="Joint_3"
+    type="revolute">
+    <origin
+      xyz="0.0318000000000006 0 0.1125"
+      rpy="0 0.00119783187528121 0" />
+    <parent
+      link="Link_2" />
+    <child
+      link="Link_3" />
+    <axis
+      xyz="0 1 0" />
+    <limit
+      lower="-1.57"
+      upper="1.57"
+      effort="2.94"
+      velocity="4.5" />
+  </joint>
+  <link
+    name="Link_4">
+    <inertial>
+      <origin
+        xyz="0.0207195207783508 0.00250991429287713 0.00203821404721022"
+        rpy="0 0 0" />
+      <mass
+        value="0.0337528735584262" />
+      <inertia
+        ixx="5.16898889782868E-06"
+        ixy="-4.30565260535002E-09"
+        ixz="4.70490364581223E-08"
+        iyy="4.01910605691164E-06"
+        iyz="5.61146571756272E-08"
+        izz="3.87872394301694E-06" />
+    </inertial>
+    <visual>
+      <origin
+        xyz="0 0 0"
+        rpy="0 0 0" />
+      <geometry>
+        <mesh
+          filename="package://arm_description/meshes/Link_4.STL" />
+      </geometry>
+      <material
+        name="">
+        <color
+          rgba="0.752941176470588 0.752941176470588 0.752941176470588 1" />
+      </material>
+    </visual>
+    <collision>
+      <origin
+        xyz="0 0 0"
+        rpy="0 0 0" />
+      <geometry>
+        <mesh
+          filename="package://arm_description/meshes/Link_4.STL" />
+      </geometry>
+    </collision>
+  </link>
+  <joint
+    name="Joint_4"
+    type="revolute">
+    <origin
+      xyz="0.1378 0 0.00016506"
+      rpy="0 -0.0011978 0" />
+    <parent
+      link="Link_3" />
+    <child
+      link="Link_4" />
+    <axis
+      xyz="0 1 0" />
+    <limit
+      lower="-1.57"
+      upper="1.57"
+      effort="2.94"
+      velocity="4.5" />
+  </joint>
+  <link
+    name="Link_5">
+    <inertial>
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
File: install/arm_description/share/arm_description/urdf/arm.urdf.xacro (robot description, xacro)
@@ -1,115 +1 @@
-<?xml version="1.0"?>
-<robot name="six_servo_arm" xmlns:xacro="http://www.ros.org/wiki/xacro">
-  <!-- Placeholder dimensions, in meters -->
-  <xacro:property name="base_h" value="0.06"/>
-  <xacro:property name="upper_arm" value="0.12"/>
-  <xacro:property name="forearm" value="0.12"/>
-  <xacro:property name="wrist_len" value="0.06"/>
-  <!-- Reusable visual link -->
-  <xacro:macro name="arm_link" params="name length radius">
-    <link name="${name}">
-      <visual>
-        <origin xyz="0 0 ${length/2}" rpy="0 0 0"/>
-        <geometry>
-          <cylinder radius="${radius}" length="${length}"/>
-        </geometry>
-        <material name="arm_blue">
-          <color rgba="0.2 0.4 0.8 1"/>
-        </material>
-      </visual>
-      <collision>
-        <origin xyz="0 0 ${length/2}"/>
-        <geometry>
-          <cylinder radius="${radius}" length="${length}"/>
-        </geometry>
-      </collision>
-      <inertial>
-        <origin xyz="0 0 ${length/2}"/>
-        <mass value="0.2"/>
-        <inertia ixx="0.001" ixy="0" ixz="0"
-                 iyy="0.001" iyz="0" izz="0.001"/>
-      </inertial>
-    </link>
-  </xacro:macro>
-  <!-- Base -->
-  <link name="base_link">
-    <visual>
-      <geometry>
-        <cylinder radius="0.055" length="${base_h}"/>
-      </geometry>
-      <material name="base_gray">
-        <color rgba="0.35 0.35 0.35 1"/>
-      </material>
-    </visual>
-    <collision>
-      <geometry>
-        <cylinder radius="0.055" length="${base_h}"/>
-      </geometry>
-    </collision>
-    <inertial>
-      <mass value="1.0"/>
-      <inertia ixx="0.002" ixy="0" ixz="0"
-               iyy="0.002" iyz="0" izz="0.002"/>
-    </inertial>
-  </link>
-  <!-- Servo 1: base rotation -->
-  <link name="shoulder_mount">
-    <visual>
-      <geometry><cylinder radius="0.035" length="0.04"/></geometry>
-      <material name="joint_gray">
-        <color rgba="0.5 0.5 0.5 1"/></material>
-    </visual>
-  </link>
-  <joint name="base_yaw" type="revolute">
-    <parent link="base_link"/>
-    <child link="shoulder_mount"/>
-    <origin xyz="0 0 ${base_h/2}" rpy="0 0 0"/>
-    <axis xyz="0 0 1"/>
-    <limit lower="-2.35" upper="2.35" effort="5" velocity="1.0"/>
-  </joint>
-  <!-- Servo 2: shoulder pitch -->
-  <xacro:arm_link name="upper_arm_link" length="${upper_arm}" radius="0.018"/>
-  <joint name="shoulder_pitch" type="revolute">
-    <parent link="shoulder_mount"/>
-    <child link="upper_arm_link"/>
-    <origin xyz="0 0 0.02" rpy="0 0 0"/>
-    <axis xyz="0 1 0"/>
-    <limit lower="-1.57" upper="1.57" effort="5" velocity="1.0"/>
-  </joint>
-  <!-- Servo 3: elbow pitch -->
-  <xacro:arm_link name="forearm_link" length="${forearm}" radius="0.015"/>
-  <joint name="elbow_pitch" type="revolute">
-    <parent link="upper_arm_link"/>
-    <child link="forearm_link"/>
-    <origin xyz="0 0 ${upper_arm}" rpy="0 0 0"/>
-    <axis xyz="0 1 0"/>
-    <limit lower="-2.0" upper="2.0" effort="5" velocity="1.0"/>
-  </joint>
-  <!-- Servo 4: wrist pitch -->
-  <xacro:arm_link name="wrist_pitch_link" length="${wrist_len}" radius="0.012"/>
-  <joint name="wrist_pitch" type="revolute">
-    <parent link="forearm_link"/>
-    <child link="wrist_pitch_link"/>
-    <origin xyz="0 0 ${forearm}" rpy="0 0 0"/>
-    <axis xyz="0 1 0"/>
-    <limit lower="-1.57" upper="1.57" effort="3" velocity="1.0"/>
-  </joint>
-  <!-- Servo 5: wrist rotation -->
-  <link name="gripper_mount"/>
-  <joint name="wrist_roll" type="revolute">
-    <parent link="wrist_pitch_link"/>
-    <child link="gripper_mount"/>
-    <origin xyz="0 0 ${wrist_len}" rpy="0 0 0"/>
-    <axis xyz="0 0 1"/>
-    <limit lower="-2.35" upper="2.35" effort="3" velocity="1.0"/>
-  </joint>
-  <!-- Servo 6: gripper opening -->
-  <xacro:arm_link name="gripper_finger" length="0.05" radius="0.005"/>
-  <joint name="gripper" type="revolute">
-    <parent link="gripper_mount"/>
-    <child link="gripper_finger"/>
-    <origin xyz="0 0 0.025" rpy="0 0 0"/>
-    <axis xyz="1 0 0"/>
-    <limit lower="0" upper="0.7" effort="2" velocity="1.0"/>
-  </joint>
-</robot>
+/root/Capstone/AMD-Capstone/arm_description/urdf/arm.urdf.xacro

Commit message: Arm is able to generate in Gazebo

File: arm_description/urdf/arm.urdf.xacro (robot description, xacro)
@@ -1,6 +1,3 @@
 <?xml version="1.0" encoding="utf-8"?>
-<!-- This URDF was automatically created by SolidWorks to URDF Exporter! Originally created by Stephen Brawner (brawner@gmail.com)
-     Commit Version: 1.6.0-4-g7f85cfe  Build Version: 1.6.7995.38578
-     For more information, please see http://wiki.ros.org/sw_urdf_exporter -->
 <robot
   name="arm_description">
@@ -485,3 +482,48 @@
       velocity="4.5" />
   </joint>
+  <ros2_control name="GazeboSystem" type="system">
+    <hardware>
+      <plugin>gazebo_ros2_control/GazeboSystem</plugin>
+    </hardware>
+    <joint name="Joint_1">
+      <command_interface name="position"/>
+      <state_interface name="position"/>
+      <state_interface name="velocity"/>
+    </joint>
+    <joint name="Joint_2">
+      <command_interface name="position"/>
+      <state_interface name="position"/>
+      <state_interface name="velocity"/>
+    </joint>
+    <joint name="Joint_3">
+      <command_interface name="position"/>
+      <state_interface name="position"/>
+      <state_interface name="velocity"/>
+    </joint>
+    <joint name="Joint_4">
+      <command_interface name="position"/>
+      <state_interface name="position"/>
+      <state_interface name="velocity"/>
+    </joint>
+    <joint name="Joint_5">
+      <command_interface name="position"/>
+      <state_interface name="position"/>
+      <state_interface name="velocity"/>
+    </joint>
+    <joint name="Joint_6">
+      <command_interface name="position"/>
+      <state_interface name="position"/>
+      <state_interface name="velocity"/>
+    </joint>
+    <joint name="Joint_Gripper">
+      <command_interface name="position"/>
+      <state_interface name="position"/>
+      <state_interface name="velocity"/>
+    </joint>
+  </ros2_control>
+  <gazebo>
+    <plugin filename="libgazebo_ros2_control.so" name="gazebo_ros2_control">
+      <parameters>$(find arm_description)/config/controllers.yaml</parameters>
+    </plugin>
+  </gazebo>
 </robot>

Commit message: Changed base joint to have continous rotation.

File: arm_description/urdf/arm.urdf.xacro (robot description, xacro)
@@ -90,5 +90,5 @@
   <joint
     name="Joint_1"
-    type="revolute">
+    type="continuous">
     <origin
       xyz="0 0 0.0520999749999999"
@@ -101,6 +101,4 @@
       xyz="0 0 1" />
     <limit
-      lower="-3.14"
-      upper="3.14"
       effort="2.92"
       velocity="4.5" />
@@ -217,6 +215,6 @@
       xyz="0 1 0" />
     <limit
-      lower="-1.57"
-      upper="1.57"
+      lower="-2.10"
+      upper="2.10"
       effort="2.94"
       velocity="4.5" />
@@ -322,5 +320,5 @@
   <joint
     name="Joint_5"
-    type="revolute">
+    type="fixed">
     <origin
       xyz="0.0344999999999794 0 0"
@@ -330,11 +328,4 @@
     <child
       link="Link_5" />
-    <axis
-      xyz="0 0 1" />
-    <limit
-      lower="-1.46"
-      upper="1.57"
-      effort="2.92"
-      velocity="4.5" />
   </joint>
   <link
@@ -506,9 +497,4 @@
       <state_interface name="velocity"/>
     </joint>
-    <joint name="Joint_5">
-      <command_interface name="position"/>
-      <state_interface name="position"/>
-      <state_interface name="velocity"/>
-    </joint>
     <joint name="Joint_6">
       <command_interface name="position"/>

Commit message: Basic arm movement working for pick and place. Need to increase force on gripper.

File: arm_description/urdf/arm.urdf.xacro (robot description, xacro)
@@ -472,4 +472,6 @@
       effort="2.92"
       velocity="4.5" />
+    <dynamics damping="0.02"/>
+    <limit lower="-0.5" upper="0.18" effort="2.92" velocity="4.5"/>
   </joint>
   <ros2_control name="GazeboSystem" type="system">
@@ -503,5 +505,7 @@
     </joint>
     <joint name="Joint_Gripper">
-      <command_interface name="position"/>
+      <command_interface name="effort">
+        <param name="min">-1</param><param name="max">1</param>
+      </command_interface>
       <state_interface name="position"/>
       <state_interface name="velocity"/>
@@ -523,3 +527,8 @@
     <minDepth>0.001</minDepth>
   </gazebo>
+  <link name="world"/>
+    <joint name="world_fixed" type="fixed">
+    <parent link="world"/><child link="base_link"/>
+    <origin xyz="0 0 0" rpy="0 0 0"/>
+  </joint>
 </robot>

Commit message: Arm moves, but has issue gripping test objects

File: arm_description/urdf/arm.urdf.xacro (robot description, xacro)
@@ -3,5 +3,15 @@
   name="arm_description">
   <link name="base_link">
+    <inertial>
+      <origin xyz="0 0 0" rpy="0 0 0"/>
+      <mass value="0.001"/>
+      <inertia ixx="1e-9" ixy="0" ixz="0" iyy="1e-9" iyz="0" izz="1e-9"/>
+    </inertial>
    </link>
+  <link name="world"/>
+    <joint name="world_fixed" type="fixed">
+    <parent link="world"/><child link="base_link"/>
+    <origin xyz="0 0 0" rpy="0 0 0"/>
+  </joint>
   <joint name="Base_joint" type="fixed">
      <parent link="base_link"/>
@@ -469,9 +479,9 @@
     <limit
       lower="-0.5"
-      upper="0.18"
+      upper="0.10"
       effort="2.92"
       velocity="4.5" />
     <dynamics damping="0.02"/>
-    <limit lower="-0.5" upper="0.18" effort="2.92" velocity="4.5"/>
+    <limit lower="-0.5" upper="0.10" effort="2.92" velocity="4.5"/>
   </joint>
   <ros2_control name="GazeboSystem" type="system">
@@ -518,17 +528,12 @@
   </gazebo>
   <gazebo reference="Gripper">
-    <mu1>1.0</mu1><mu2>1.0</mu2>
+    <mu1>10.0</mu1><mu2>10.0</mu2>
     <kp>1e5</kp><kd>10</kd>
     <minDepth>0.001</minDepth>
   </gazebo>
   <gazebo reference="Link_6">
-    <mu1>1.0</mu1><mu2>1.0</mu2>
+    <mu1>10.0</mu1><mu2>10.0</mu2>
     <kp>1e5</kp><kd>10</kd>
     <minDepth>0.001</minDepth>
   </gazebo>
-  <link name="world"/>
-    <joint name="world_fixed" type="fixed">
-    <parent link="world"/><child link="base_link"/>
-    <origin xyz="0 0 0" rpy="0 0 0"/>
-  </joint>
 </robot>
