Commit message: New meshes working on arm. Gripper needs to be added.

File: arm_description/urdf/arm.urdf.xacro (robot description, xacro)
@@ -1,539 +1,4 @@
-<?xml version="1.0" encoding="utf-8"?>
-<robot
-  name="arm_description">
-  <link name="base_link">
-    <inertial>
-      <origin xyz="0 0 0" rpy="0 0 0"/>
-      <mass value="0.001"/>
-      <inertia ixx="1e-9" ixy="0" ixz="0" iyy="1e-9" iyz="0" izz="1e-9"/>
-    </inertial>
-   </link>
-  <link name="world"/>
-    <joint name="world_fixed" type="fixed">
-    <parent link="world"/><child link="base_link"/>
-    <origin xyz="0 0 0" rpy="0 0 0"/>
-  </joint>
-  <joint name="Base_joint" type="fixed">
-     <parent link="base_link"/>
-     <child link="Link_0"/>
-   </joint>
-  <link
-    name="Link_0">
-    <inertial>
-      <origin
-        xyz="-0.00186841174166371 2.50538852245872E-08 0.0215517174968573"
-        rpy="0 0 0" />
-      <mass
-        value="0.120274881687953" />
-      <inertia
-        ixx="7.85095489782459E-05"
-        ixy="-2.5923964914073E-10"
-        ixz="7.52479004938925E-07"
-        iyy="5.40736714848378E-05"
-        iyz="-1.15213465229022E-10"
-        izz="0.000105809384793902" />
-    </inertial>
-    <visual>
-      <origin
-        xyz="0 0 0"
-        rpy="0 0 0" />
-      <geometry>
-        <mesh
-          filename="package://arm_description/meshes/Link_0.STL" />
-      </geometry>
-      <material
-        name="">
-        <color
-          rgba="0.752941176470588 0.752941176470588 0.752941176470588 1" />
-      </material>
-    </visual>
-    <collision>
-      <origin
-        xyz="0 0 0"
-        rpy="0 0 0" />
-      <geometry>
-        <mesh
-          filename="package://arm_description/meshes/Link_0.STL" />
-      </geometry>
-    </collision>
-  </link>
-  <link
-    name="Link_1">
-    <inertial>
-      <origin
-        xyz="1.6372825671052E-08 -0.00192246981351583 0.0249618879819944"
-        rpy="0 0 0" />
-      <mass
-        value="0.0601843511838218" />
-      <inertia
-        ixx="2.40354508371122E-05"
-        ixy="7.39479891402167E-12"
-        ixz="2.05889155998936E-11"
-        iyy="2.50929356191337E-05"
-        iyz="-2.8998043123432E-07"
-        izz="1.79760286790951E-05" />
-    </inertial>
-    <visual>
-      <origin
-        xyz="0 0 0"
-        rpy="0 0 0" />
-      <geometry>
-        <mesh
-          filename="package://arm_description/meshes/Link_1.STL" />
-      </geometry>
-      <material
-        name="">
-        <color
-          rgba="0.752941176470588 0.752941176470588 0.752941176470588 1" />
-      </material>
-    </visual>
-    <collision>
-      <origin
-        xyz="0 0 0"
-        rpy="0 0 0" />
-      <geometry>
-        <mesh
-          filename="package://arm_description/meshes/Link_1.STL" />
-      </geometry>
-    </collision>
-  </link>
-  <joint
-    name="Joint_1"
-    type="continuous">
-    <origin
-      xyz="0 0 0.0520999749999999"
-      rpy="0 0 0" />
-    <parent
-      link="Link_0" />
-    <child
-      link="Link_1" />
-    <axis
-      xyz="0 0 1" />
-    <limit
-      effort="2.92"
-      velocity="4.5" />
-  </joint>
-  <link
-    name="Link_2">
-    <inertial>
-      <origin
-        xyz="0.00639934747655226 -0.000788371670941635 0.0673431569215511"
-        rpy="0 0 0" />
-      <mass
-        value="0.0879365609479581" />
-      <inertia
-        ixx="5.58125584142004E-05"
-        ixy="3.05873895421976E-07"
-        ixz="-6.11348651523486E-07"
-        iyy="5.08744603129432E-05"
-        iyz="2.78428454591459E-07"
-        izz="2.91228934054131E-05" />
-    </inertial>
-    <visual>
-      <origin
-        xyz="0 0 0"
-        rpy="0 0 0" />
-      <geometry>
-        <mesh
-          filename="package://arm_description/meshes/Link_2.STL" />
-      </geometry>
-      <material
-        name="">
-        <color
-          rgba="0.752941176470588 0.752941176470588 0.752941176470588 1" />
-      </material>
-    </visual>
-    <collision>
-      <origin
-        xyz="0 0 0"
-        rpy="0 0 0" />
-      <geometry>
-        <mesh
-          filename="package://arm_description/meshes/Link_2.STL" />
-      </geometry>
-    </collision>
-  </link>
-  <joint
-    name="Joint_2"
-    type="revolute">
-    <origin
-      xyz="0 0 0.0541000250000002"
-      rpy="0 0 0" />
-    <parent
-      link="Link_1" />
-    <child
-      link="Link_2" />
-    <axis
-      xyz="0 1 0" />
-    <limit
-      lower="-1.57"
-      upper="1.57"
-      effort="2.94"
-      velocity="4.5" />
-  </joint>
-  <link
-    name="Link_3">
-    <inertial>
-      <origin
-        xyz="0.0717174331065269 -0.000795514048423572 0.000196159539195329"
-        rpy="0 0 0" />
-      <mass
-        value="0.0879996844183864" />
-      <inertia
-        ixx="2.19988198885556E-05"
-        ixy="5.11334783735054E-07"
-        ixz="-2.57342143473836E-08"
-        iyy="5.13996982896891E-05"
-        iyz="5.45466342941832E-11"
-        izz="6.34682921546949E-05" />
-    </inertial>
-    <visual>
-      <origin
-        xyz="0 0 0"
-        rpy="0 0 0" />
-      <geometry>
-        <mesh
-          filename="package://arm_description/meshes/Link_3.STL" />
-      </geometry>
-      <material
-        name="">
-        <color
-          rgba="0.752941176470588 0.752941176470588 0.752941176470588 1" />
-      </material>
-    </visual>
-    <collision>
-      <origin
-        xyz="0 0 0"
-        rpy="0 0 0" />
-      <geometry>
-        <mesh
-          filename="package://arm_description/meshes/Link_3.STL" />
-      </geometry>
-    </collision>
-  </link>
-  <joint
-    name="Joint_3"
-    type="revolute">
-    <origin
-      xyz="0.0318000000000006 0 0.1125"
-      rpy="0 0.00119783187528121 0" />
-    <parent
-      link="Link_2" />
-    <child
-      link="Link_3" />
-    <axis
-      xyz="0 1 0" />
-    <limit
-      lower="-2.10"
-      upper="2.10"
-      effort="2.94"
-      velocity="4.5" />
-  </joint>
-  <link
-    name="Link_4">
-    <inertial>
-      <origin
-        xyz="0.0207195207783508 0.00250991429287713 0.00203821404721022"
-        rpy="0 0 0" />
-      <mass
-        value="0.0337528735584262" />
-      <inertia
-        ixx="5.16898889782868E-06"
-        ixy="-4.30565260535002E-09"
-        ixz="4.70490364581223E-08"
-        iyy="4.01910605691164E-06"
-        iyz="5.61146571756272E-08"
-        izz="3.87872394301694E-06" />
-    </inertial>
-    <visual>
-      <origin
-        xyz="0 0 0"
-        rpy="0 0 0" />
-      <geometry>
-        <mesh
-          filename="package://arm_description/meshes/Link_4.STL" />
-      </geometry>
-      <material
-        name="">
-        <color
-          rgba="0.752941176470588 0.752941176470588 0.752941176470588 1" />
-      </material>
-    </visual>
-    <collision>
-      <origin
-        xyz="0 0 0"
-        rpy="0 0 0" />
-      <geometry>
-        <mesh
-          filename="package://arm_description/meshes/Link_4.STL" />
-      </geometry>
-    </collision>
-  </link>
-  <joint
-    name="Joint_4"
-    type="revolute">
-    <origin
-      xyz="0.1378 0 0.00016506"
-      rpy="0 -0.0011978 0" />
-    <parent
-      link="Link_3" />
-    <child
-      link="Link_4" />
-    <axis
-      xyz="0 1 0" />
-    <limit
-      lower="-1.57"
-      upper="1.57"
-      effort="2.94"
-      velocity="4.5" />
-  </joint>
-  <link
-    name="Link_5">
-    <inertial>
-      <origin
-        xyz="0.0240131840829411 2.71687309323209E-07 0.0187123881058747"
-        rpy="0 0 0" />
-      <mass
-        value="0.0567730043412737" />
-      <inertia
-        ixx="1.64904144549218E-05"
-        ixy="-6.16564440638043E-11"
-        ixz="1.61324277303039E-06"
-        iyy="2.43462036741009E-05"
-        iyz="2.75698618885409E-10"
-        izz="2.39782654452867E-05" />
-    </inertial>
-    <visual>
-      <origin
-        xyz="0 0 0"
-        rpy="0 0 0" />
-      <geometry>
-        <mesh
-          filename="package://arm_description/meshes/Link_5.STL" />
-      </geometry>
-      <material
-        name="">
-        <color
-          rgba="0.752941176470588 0.752941176470588 0.752941176470588 1" />
-      </material>
-    </visual>
-    <collision>
-      <origin
-        xyz="0 0 0"
-        rpy="0 0 0" />
-      <geometry>
-        <mesh
-          filename="package://arm_description/meshes/Link_5.STL" />
-      </geometry>
-    </collision>
-  </link>
-  <joint
-    name="Joint_5"
-    type="fixed">
-    <origin
-      xyz="0.0344999999999794 0 0"
-      rpy="0 0 0" />
-    <parent
-      link="Link_4" />
-    <child
-      link="Link_5" />
-  </joint>
-  <link
-    name="Link_6">
-    <inertial>
-      <origin
-        xyz="0.0257518935612762 0.00281937583164617 0.00493977898472961"
-        rpy="0 0 0" />
-      <mass
-        value="0.0319894081273108" />
-      <inertia
-        ixx="1.31065564223499E-05"
-        ixy="-3.37815187638791E-07"
-        ixz="2.09094384952868E-06"
-        iyy="1.53996224639332E-05"
-        iyz="5.58847684910504E-07"
-        izz="8.92019679064812E-06" />
-    </inertial>
-    <visual>
-      <origin
-        xyz="0 0 0"
-        rpy="0 0 0" />
-      <geometry>
-        <mesh
-          filename="package://arm_description/meshes/Link_6.STL" />
-      </geometry>
-      <material
-        name="">
-        <color
-          rgba="0.752941176470588 0.752941176470588 0.752941176470588 1" />
-      </material>
-    </visual>
-    <collision>
-      <origin
-        xyz="0 0 0"
-        rpy="0 0 0" />
-      <geometry>
-        <mesh
-          filename="package://arm_description/meshes/Link_6.STL" />
-      </geometry>
-    </collision>
-  </link>
-  <joint
-    name="Joint_6"
-    type="revolute">
-    <origin
-      xyz="0.0576950428676977 0 -0.00754999999999195"
-      rpy="0 0 0" />
-    <parent
-      link="Link_5" />
-    <child
-      link="Link_6" />
-    <axis
-      xyz="1 0 0" />
-    <limit
-      lower="-3.14"
-      upper="3.14"
-      effort="2.94"
-      velocity="4.5" />
-  </joint>
-  <link
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