Commit message: Added new mesh into Moveit2 controller

File: arm_description/urdf/new_arm.urdf.xacro (robot description, xacro)
@@ -164,28 +164,40 @@
     <limit effort="2.94" lower="-1.57" upper="1.57" velocity="0.5"/>
   </joint>
-  <joint name="Joint_Gripper" type="fixed">
+  <joint name="Joint_Gripper" type="revolute">
   <parent link="hand_link"/><child link="grip_left_link"/>
-  <origin rpy="-1.57 0 0" xyz="0 0.015 0.030"/>
-</joint>
-<joint name="grip_right" type="fixed">
-  <parent link="hand_link"/><child link="grip_right_link"/>
-  <origin rpy="1.57 0 0" xyz="0 -0.015 0.030"/>
-</joint>
-<joint name="tendon_left" type="fixed">
-  <parent link="hand_link"/><child link="tendon_left_link"/>
-  <origin rpy="-1.57 0 0" xyz="0 0.005 0.050"/>
-</joint>
-<joint name="tendon_right" type="fixed">
-  <parent link="hand_link"/><child link="tendon_right_link"/>
-  <origin rpy="1.57 0 0" xyz="0 -0.005 0.050"/>
-</joint>
-<joint name="finger_left" type="fixed">
-  <parent link="grip_left_link"/><child link="finger_left_link"/>
-  <origin rpy="1.57 0 0" xyz="0 0 0.030"/>
-</joint>
-<joint name="finger_right" type="fixed">
-  <parent link="grip_right_link"/><child link="finger_right_link"/>
-  <origin rpy="-1.57 0 0" xyz="0 0 0.030"/>
-</joint>
+  <origin rpy="-1.57 0 0" xyz="0 0.015 0.030"/><axis xyz="-1 0 0"/>
+  <limit effort="1.0" lower="-1.57" upper="0" velocity="0.5"/>
+  <dynamics damping="0.02"/>
+  </joint>
+  <joint name="grip_right" type="revolute">
+    <parent link="hand_link"/><child link="grip_right_link"/>
+    <origin rpy="1.57 0 0" xyz="0 -0.015 0.030"/><axis xyz="-1 0 0"/>
+    <limit effort="1.0" lower="0" upper="1.57" velocity="0.5"/>
+    <dynamics damping="0.02"/>
+  </joint>
+  <joint name="tendon_left" type="revolute">
+    <parent link="hand_link"/><child link="tendon_left_link"/>
+    <origin rpy="-1.57 0 0" xyz="0 0.005 0.050"/><axis xyz="-1 0 0"/>
+    <limit effort="1.0" lower="-1.57" upper="0" velocity="0.5"/>
+    <dynamics damping="0.02"/>
+  </joint>
+  <joint name="tendon_right" type="revolute">
+    <parent link="hand_link"/><child link="tendon_right_link"/>
+    <origin rpy="1.57 0 0" xyz="0 -0.005 0.050"/><axis xyz="-1 0 0"/>
+    <limit effort="1.0" lower="0" upper="1.57" velocity="0.5"/>
+    <dynamics damping="0.02"/>
+  </joint>
+  <joint name="finger_left" type="revolute">
+    <parent link="grip_left_link"/><child link="finger_left_link"/>
+    <origin rpy="1.57 0 0" xyz="0 0 0.030"/><axis xyz="-1 0 0"/>
+    <limit effort="1.0" lower="0" upper="1.57" velocity="0.5"/>
+    <dynamics damping="0.02"/>
+  </joint>
+  <joint name="finger_right" type="revolute">
+    <parent link="grip_right_link"/><child link="finger_right_link"/>
+    <origin rpy="-1.57 0 0" xyz="0 0 0.030"/><axis xyz="-1 0 0"/>
+    <limit effort="1.0" lower="-1.57" upper="0" velocity="0.5"/>
+    <dynamics damping="0.02"/>
+  </joint>
   <joint name="EE_Gripper_Joint" type="fixed">
     <parent link="hand_link"/><child link="EE_Gripper_Link"/>
@@ -214,4 +226,10 @@
       <state_interface name="position"/><state_interface name="velocity"/>
     </joint>
+    <joint name="Joint_Gripper"><command_interface name="position"/><state_interface name="position"/><state_interface name="velocity"/></joint>
+    <joint name="grip_right"><command_interface name="position"/><state_interface name="position"/><state_interface name="velocity"/></joint>
+    <joint name="tendon_left"><command_interface name="position"/><state_interface name="position"/><state_interface name="velocity"/></joint>
+    <joint name="tendon_right"><command_interface name="position"/><state_interface name="position"/><state_interface name="velocity"/></joint>
+    <joint name="finger_left"><command_interface name="position"/><state_interface name="position"/><state_interface name="velocity"/></joint>
+    <joint name="finger_right"><command_interface name="position"/><state_interface name="position"/><state_interface name="velocity"/></joint>
   </ros2_control>
   <gazebo>

Commit message: Updated single arm simulation

File: arm_description/urdf/new_arm.urdf.xacro (robot description, xacro)
@@ -16,4 +16,5 @@
       <origin xyz="0 0 0.006903"/>
       <geometry><mesh filename="package://arm_description/meshes/base.stl"/></geometry>
+      <material name="base_slate"><color rgba="0.22 0.27 0.32 1"/></material>
     </visual>
     <collision>
@@ -29,5 +30,8 @@
                iyy="0.000032568110" iyz="0" izz="0.000052867674"/>
     </inertial>
-    <visual><geometry><mesh filename="package://arm_description/meshes/shoulder.stl"/></geometry></visual>
+    <visual>
+      <geometry><mesh filename="package://arm_description/meshes/shoulder.stl"/></geometry>
+      <material name="shoulder_blue"><color rgba="0.12 0.35 0.72 1"/></material>
+    </visual>
     <collision><geometry><mesh filename="package://arm_description/meshes/shoulder.stl"/></geometry></collision>
   </link>
@@ -39,5 +43,8 @@
                iyy="0.000027964460" iyz="0" izz="0.000006091413"/>
     </inertial>
-    <visual><geometry><mesh filename="package://arm_description/meshes/humerus.stl"/></geometry></visual>
+    <visual>
+      <geometry><mesh filename="package://arm_description/meshes/humerus.stl"/></geometry>
+      <material name="humerus_orange"><color rgba="0.92 0.35 0.10 1"/></material>
+    </visual>
     <collision><geometry><mesh filename="package://arm_description/meshes/humerus.stl"/></geometry></collision>
   </link>
@@ -49,5 +56,8 @@
                iyy="0.000045024344" iyz="0" izz="0.000013082564"/>
     </inertial>
-    <visual><geometry><mesh filename="package://arm_description/meshes/forearm.stl"/></geometry></visual>
+    <visual>
+      <geometry><mesh filename="package://arm_description/meshes/forearm.stl"/></geometry>
+      <material name="forearm_teal"><color rgba="0.05 0.58 0.52 1"/></material>
+    </visual>
     <collision><geometry><mesh filename="package://arm_description/meshes/forearm.stl"/></geometry></collision>
   </link>
@@ -59,5 +69,8 @@
                iyy="0.000021977992" iyz="0" izz="0.000014241720"/>
     </inertial>
-    <visual><geometry><mesh filename="package://arm_description/meshes/wrist.stl"/></geometry></visual>
+    <visual>
+      <geometry><mesh filename="package://arm_description/meshes/wrist.stl"/></geometry>
+      <material name="wrist_gold"><color rgba="0.92 0.68 0.12 1"/></material>
+    </visual>
     <collision><geometry><mesh filename="package://arm_description/meshes/wrist.stl"/></geometry></collision>
   </link>
@@ -69,5 +82,8 @@
                iyy="0.000008729011" iyz="0" izz="0.000008671204"/>
     </inertial>
-    <visual><geometry><mesh filename="package://arm_description/meshes/hand.stl"/></geometry></visual>
+    <visual>
+      <geometry><mesh filename="package://arm_description/meshes/hand.stl"/></geometry>
+      <material name="hand_purple"><color rgba="0.48 0.20 0.68 1"/></material>
+    </visual>
     <collision><geometry><mesh filename="package://arm_description/meshes/hand.stl"/></geometry></collision>
   </link>
@@ -79,5 +95,8 @@
                iyy="0.000000449149" iyz="0" izz="0.000000142956"/>
     </inertial>
-    <visual><geometry><mesh filename="package://arm_description/meshes/carpal-left.stl"/></geometry></visual>
+    <visual>
+      <geometry><mesh filename="package://arm_description/meshes/carpal-left.stl"/></geometry>
+      <material name="gripper_gray"><color rgba="0.38 0.42 0.47 1"/></material>
+    </visual>
     <collision><geometry><mesh filename="package://arm_description/meshes/carpal-left.stl"/></geometry></collision>
   </link>
@@ -89,5 +108,8 @@
                iyy="0.000000568082" iyz="0" izz="0.000000191833"/>
     </inertial>
-    <visual><geometry><mesh filename="package://arm_description/meshes/carpal-right.stl"/></geometry></visual>
+    <visual>
+      <geometry><mesh filename="package://arm_description/meshes/carpal-right.stl"/></geometry>
+      <material name="gripper_gray"><color rgba="0.38 0.42 0.47 1"/></material>
+    </visual>
     <collision><geometry><mesh filename="package://arm_description/meshes/carpal-right.stl"/></geometry></collision>
   </link>
@@ -99,5 +121,8 @@
                iyy="0.000000093216" iyz="0" izz="0.000000012587"/>
     </inertial>
-    <visual><geometry><mesh filename="package://arm_description/meshes/tendon.stl"/></geometry></visual>
+    <visual>
+      <geometry><mesh filename="package://arm_description/meshes/tendon.stl"/></geometry>
+      <material name="tendon_dark"><color rgba="0.16 0.18 0.20 1"/></material>
+    </visual>
     <collision><geometry><mesh filename="package://arm_description/meshes/tendon.stl"/></geometry></collision>
   </link>
@@ -109,5 +134,8 @@
                iyy="0.000000093216" iyz="0" izz="0.000000012587"/>
     </inertial>
-    <visual><geometry><mesh filename="package://arm_description/meshes/tendon.stl"/></geometry></visual>
+    <visual>
+      <geometry><mesh filename="package://arm_description/meshes/tendon.stl"/></geometry>
+      <material name="tendon_dark"><color rgba="0.16 0.18 0.20 1"/></material>
+    </visual>
     <collision><geometry><mesh filename="package://arm_description/meshes/tendon.stl"/></geometry></collision>
   </link>
@@ -119,5 +147,8 @@
                iyy="0.000000890885" iyz="0" izz="0.000000113650"/>
     </inertial>
-    <visual><geometry><mesh filename="package://arm_description/meshes/finger.stl"/></geometry></visual>
+    <visual>
+      <geometry><mesh filename="package://arm_description/meshes/finger.stl"/></geometry>
+      <material name="finger_blue"><color rgba="0.18 0.48 0.78 1"/></material>
+    </visual>
     <collision><geometry><mesh filename="package://arm_description/meshes/finger.stl"/></geometry></collision>
   </link>
@@ -132,4 +163,5 @@
       <origin rpy="0 0 3.14159"/>
       <geometry><mesh filename="package://arm_description/meshes/finger.stl"/></geometry>
+      <material name="finger_blue"><color rgba="0.18 0.48 0.78 1"/></material>
     </visual>
     <collision>
